Commit message: fix simulation and add mycobot arm

File: src/limo_manipulator_description/urdf/limo_manipulator.xacro (robot description, xacro)
@@ -1,37 +1,58 @@
 <?xml version="1.0"?>
 <robot name="limo_manipulator" xmlns:xacro="http://ros.org/wiki/xacro">
-  <!-- Include Limo Robot -->
+  <!-- ================================================================
+       arm_type: "open_manipulator" | "mycobot" | "none"
+       Selects which manipulator arm to mount on the LIMO chassis.
+       ================================================================ -->
+  <xacro:arg name="arm_type" default="open_manipulator"/>
+  <xacro:property name="arm_type" value="$(arg arm_type)"/>
+  <!-- ======================== LIMO Base ============================ -->
   <xacro:include filename="$(find limo_description)/urdf/limo_four_diff.xacro" />
-  <!-- Include OpenManipulator-X -->
-  <xacro:include filename="$(find open_manipulator_description)/urdf/open_manipulator_x/open_manipulator_x_arm.urdf.xacro" />
-  <xacro:include filename="$(find open_manipulator_description)/gazebo/open_manipulator_x.gazebo.xacro" />
-  <!-- Include our custom ros2_control for the arm -->
-  <xacro:include filename="$(find limo_manipulator_description)/urdf/manipulator_control.ros2_control.xacro" />
-  <!-- Attachment point for the manipulator.
-       LIMO chassis dimensions: base_z_size=0.10 m centered at base_link.
-       Top surface of chassis is at z=+0.05 m from base_link.
-       The arm is bolted on the front-top plate, so z=+0.05.
-       x=0.04 m forward keeps the arm centred over the front half of the chassis. -->
-  <joint name="manipulator_mounting_joint" type="fixed">
-    <parent link="base_link" />
-    <child link="link1" />
-    <origin xyz="0.04 0.0 0.05" rpy="0 0 0" />
-  </joint>
-  <!-- OpenManipulator-X Arm Macro -->
-  <xacro:open_manipulator_x prefix="" />
-  <!-- Gazebo properties for OpenManipulator -->
-  <xacro:open_manipulator_x_gazebo prefix="" />
-  <!-- Integrated ros2_control hardware interface for the arm -->
-  <xacro:limo_manipulator_control prefix="" />
-  <!-- Gazebo Sim Plugins -->
+  <!-- ======================== OpenManipulator-X ==================== -->
+  <xacro:if value="${arm_type == 'open_manipulator'}">
+    <xacro:include filename="$(find open_manipulator_x_description)/urdf/open_manipulator_x_arm.urdf.xacro" />
+    <xacro:include filename="$(find open_manipulator_x_description)/gazebo/open_manipulator_x.gazebo.xacro" />
+    <xacro:include filename="$(find limo_manipulator_description)/urdf/manipulator_control.ros2_control.xacro" />
+    <joint name="manipulator_mounting_joint" type="fixed">
+      <parent link="base_link" />
+      <child link="link1" />
+      <origin xyz="0.04 0.0 0.05" rpy="0 0 0" />
+    </joint>
+    <xacro:open_manipulator_x prefix="" />
+    <xacro:open_manipulator_x_gazebo prefix="" />
+    <xacro:limo_manipulator_control prefix="" />
+  </xacro:if>
+  <!-- ======================== MyCobot 280 ========================== -->
+  <xacro:if value="${arm_type == 'mycobot'}">
+    <xacro:include filename="$(find mycobot_description)/urdf/mycobot_280_arduino/mycobot_280_arduino.urdf" />
+    <xacro:include filename="$(find limo_manipulator_description)/urdf/mycobot_control.ros2_control.xacro" />
+    <joint name="manipulator_mounting_joint" type="fixed">
+      <parent link="base_link" />
+      <child link="g_base" />
+      <!-- x=0: centred on chassis, z=0.10: on top of LIMO deck (chassis top ~0.05 + base clearance) -->
+      <origin xyz="0.0 0.0 0.10" rpy="0 0 0" />
+    </joint>
+    <xacro:limo_mycobot_control prefix="" />
+  </xacro:if>
+  <!-- ======================== Gazebo Sim Plugins =================== -->
   <gazebo>
-    <plugin filename="ign_ros2_control-system" name="gz_ros2_control::GazeboSimROS2ControlPlugin">
-      <parameters>$(find limo_manipulator_bringup)/config/controllers.yaml</parameters>
-    </plugin>
-    <!-- Joint State Publisher for Gazebo Sim -->
-    <plugin filename="gz-sim-joint-state-publisher-system" name="gz::sim::systems::JointStatePublisher">
-      <topic>joint_states</topic>
-    </plugin>
-    <!-- Limo Base Diff Drive (4-wheel simplified) -->
+    <!-- ros2_control plugin (only when an arm is mounted) -->
+    <xacro:if value="${arm_type == 'open_manipulator'}">
+      <plugin filename="gz_ros2_control-system" name="gz_ros2_control::GazeboSimROS2ControlPlugin">
+        <parameters>$(find limo_manipulator_bringup)/config/controllers.yaml</parameters>
+      </plugin>
+    </xacro:if>
+    <xacro:if value="${arm_type == 'mycobot'}">
+      <plugin filename="gz_ros2_control-system" name="gz_ros2_control::GazeboSimROS2ControlPlugin">
+        <parameters>$(find limo_manipulator_bringup)/config/controllers_mycobot.yaml</parameters>
+      </plugin>
+    </xacro:if>
+    <!-- Joint State Publisher (arm joints visible to Gazebo) -->
+    <xacro:if value="${arm_type != 'none'}">
+      <plugin filename="gz-sim-joint-state-publisher-system" name="gz::sim::systems::JointStatePublisher">
+        <topic>joint_states</topic>
+      </plugin>
+    </xacro:if>
+    <!-- LIMO DiffDrive (always active, cmd_vel only, no odom) -->
     <plugin filename="gz-sim-diff-drive-system" name="gz::sim::systems::DiffDrive">
       <left_joint>front_left_wheel</left_joint>
@@ -39,23 +60,26 @@
       <right_joint>front_right_wheel</right_joint>
       <right_joint>rear_right_wheel</right_joint>
-      <wheel_separation>0.172</wheel_separation>
+      <wheel_separation>0.175</wheel_separation>
       <wheel_radius>0.045</wheel_radius>
-      <!-- 20 Hz is enough for Nav2; 50 Hz added unnecessary CPU/bus load -->
-      <odom_publish_frequency>20</odom_publish_frequency>
+      <max_linear_acceleration>1.0</max_linear_acceleration>
+      <max_angular_acceleration>2.0</max_angular_acceleration>
+      <odom_publish_frequency>0</odom_publish_frequency>
       <topic>/cmd_vel</topic>
+    </plugin>
+    <!-- Ground-truth odometry from model pose (avoids skid-steer drift) -->
+    <plugin filename="gz-sim-odometry-publisher-system" name="gz::sim::systems::OdometryPublisher">
       <odom_topic>/odom</odom_topic>
-      <tf_topic>/tf</tf_topic>
-      <frame_id>odom</frame_id>
-      <child_frame_id>base_footprint</child_frame_id>
+      <odom_frame>odom</odom_frame>
+      <robot_base_frame>base_footprint</robot_base_frame>
+      <odom_publish_frequency>30</odom_publish_frequency>
+      <dimensions>2</dimensions>
     </plugin>
   </gazebo>
-  <!-- Override Lidar for Gazebo Sim (Ignition Fortress uses gpu_lidar type) -->
-  <!-- Performance tuning:
-       - visualize=false  → no OpenGL scan-line rendering overlay in Gazebo GUI
-       - samples=360      → half resolution (1° per sample), sufficient for Nav2
-       - update_rate=8    → slightly below 10 Hz to reduce GPU lidar compute -->
+  <!-- ======================== LiDAR Sensor ========================= -->
   <gazebo reference="laser_link">
     <sensor name="laser_sensor" type="gpu_lidar">
       <topic>scan</topic>
+      <gz_frame_id>laser_link</gz_frame_id>
+      <frame_id>laser_link</frame_id>
       <update_rate>8</update_rate>
       <lidar>
@@ -78,5 +102,5 @@
     </sensor>
   </gazebo>
-  <!-- IMU for Gazebo Sim — reduced rate, no visualize -->
+  <!-- ======================== IMU Sensor =========================== -->
   <gazebo reference="imu_link">
     <sensor name="imu_sensor" type="imu">
@@ -85,12 +109,9 @@
       <visualize>false</visualize>
       <topic>imu</topic>
+      <gz_frame_id>imu_link</gz_frame_id>
+      <frame_id>imu_link</frame_id>
     </sensor>
   </gazebo>
-  <!-- ================================================================
-       RGB Camera for AprilTag detection
-       Mounted on the robot body above the arm, angled forward-down
-       to observe the workspace (tables at ~10 cm height).
-       Frame: camera_link
-       ================================================================ -->
+  <!-- ======================== RGB Camera =========================== -->
   <link name="camera_link">
     <visual>
@@ -108,24 +129,8 @@
     </inertial>
   </link>
-  <!-- Camera optical frame (Z forward, X right, Y down — ROS convention) -->
   <link name="camera_color_optical_frame"/>
   <joint name="camera_joint" type="fixed">
     <parent link="base_link"/>
     <child link="camera_link"/>
-    <!--
-      Camera is on a vertical mast, ABOVE the maximum arm reach.
-      Gazebo convention: positive pitch (rpy="0 +θ 0") tilts lens forward-down.
-      Key constraint: OpenManipulator-X max height above its base ≈ 0.38 m.
-      Mounted at z=0.05 m, the arm top is at most z ≈ 0.43 m from base_link.
-      Setting camera at z=0.52 m puts it 9 cm above maximum arm extension,
-      so the arm can NEVER enter the camera's upper FOV regardless of pose.
-      x = +0.05 m  → slightly forward of chassis centre (mast on front deck).
-      z = +0.52 m  → 52 cm above base_link ≈ 67 cm above ground. Above the
-                      tallest possible arm configuration (≈ 43 cm).
-      pitch = +50° → steeper tilt to compensate for the greater height:
-                      optical-axis at table height (0.10 m) falls
-                      ≈ 0.05 + (0.57)/tan(50°) ≈ 0.53 m in front of robot,
-                      centred on the manipulation workspace (0.3–0.8 m).
-    -->
     <origin xyz="0.05 0.0 0.52" rpy="0.0 0.873 0.0"/>
   </joint>
@@ -133,13 +138,11 @@
     <parent link="camera_link"/>
     <child link="camera_color_optical_frame"/>
-    <!-- Standard ROS optical frame rotation: z-forward, x-right, y-down -->
     <origin xyz="0 0 0" rpy="-1.5708 0 -1.5708"/>
   </joint>
-  <!-- Gazebo camera sensor (RGB) -->
   <gazebo reference="camera_link">
     <sensor name="rgb_camera" type="camera">
       <topic>camera/image_raw</topic>
       <camera>
-        <horizontal_fov>1.047</horizontal_fov>  <!-- 60 deg FOV -->
+        <horizontal_fov>1.047</horizontal_fov>
         <image>
           <width>640</width>
@@ -158,5 +161,4 @@
       </camera>
       <always_on>1</always_on>
-      <!-- 5 Hz is enough to detect AprilTags; 15 Hz causes unnecessary GPU load -->
       <update_rate>5</update_rate>
       <visualize>false</visualize>
